File: Hardware/unhappyhacking.brd (EAGLE design)
At the start: 58.4 x 50.2 mm, 19 parts, among them U1 TINY85-20-DIP

Commit message: Added firmware
Parts:
- moved R7 2.84 mm to (21.0, 17.1)
- moved U$1 2.84 mm to (31.8, 27.3)
- moved U$2 2.84 mm to (50.8, 17.8)
- moved STANDOFF4 2.84 mm to (7.62, 43.8)
- moved U$3 2.84 mm to (12.7, 27.3)
- moved STANDOFF1 2.84 mm to (7.62, 3.81)
- moved JP1 2.84 mm to (17.8, 43.8)
- moved R1 2.84 mm to (30.5, 36.2)
- moved R5 2.84 mm to (11.4, 36.2)
- moved U$4 2.84 mm to (22.2, 8.26)
- moved STANDOFF2 2.84 mm to (55.9, 3.81)
- moved R2 2.84 mm to (49.5, 26.7)
- moved STANDOFF3 2.84 mm to (55.9, 43.8)
- moved D1 2.54 mm to (35.6, 43.2)
- moved D2 2.54 mm to (39.4, 43.2)
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Routing:
- net N$6: track 23.2 -> 25.9 mm, vias 0 -> 1
- net N$2: track 25.9 -> 23.9 mm
- net RESET: track 38.1 -> 39.4 mm
- net N$3: track 25.3 -> 26.6 mm
- net MISO: track 48.0 -> 49.3 mm
- net N$7: track 26.7 -> 27.3 mm
